File: FrenGP_robot/FrenGP_robot.kicad_pcb (KiCad board)
At the start: 2 copper layers, 100 x 90 mm, 19 parts, among them J1 Screw_Terminal_01x02, J2 Screw_Terminal_01x02, J3 Screw_Terminal_01x02, SW1 SW_Push

Commit message: Update v1.1
Parts:
- removed U6, U7: ~, DRV_8833_module:3pin_Reflection_sensor
- added BZ1: Buzzer, Buzzer_Beeper:Buzzer_12x9.5RM7.6, F.Cu at (51.8, 97.2)
- added D3: LED, Diode_SMD:D_0603_1608Metric_Pad1.05x0.95mm_HandSolder, F.Cu at (58.6, 31.6)
- added D4: LED, Diode_SMD:D_0603_1608Metric_Pad1.05x0.95mm_HandSolder, F.Cu at (119.6, 108.0)
- added R2: 330R, Resistor_SMD:R_0603_1608Metric_Pad0.98x0.95mm_HandSolder, F.Cu at (52.6, 31.6)
- added R3: 0R5, Resistor_SMD:R_0805_2012Metric_Pad1.20x1.40mm_HandSolder, F.Cu at (106.9, 68.2)
- added R4: 0R5, Resistor_SMD:R_0805_2012Metric_Pad1.20x1.40mm_HandSolder, F.Cu at (94.4, 56.0)
- added R5: 330R, Resistor_SMD:R_0603_1608Metric_Pad0.98x0.95mm_HandSolder, F.Cu at (119.6, 102.0)
- added R6: 1k, Resistor_SMD:R_0603_1608Metric_Pad0.98x0.95mm_HandSolder, F.Cu at (103.5, 35.8)
- added R7: 2k, Resistor_SMD:R_0603_1608Metric_Pad0.98x0.95mm_HandSolder, F.Cu at (103.5, 32.0)
- J2: value Screw_Terminal_01x02 -> Right motor
- J3: value Screw_Terminal_01x02 -> Left motor
- R1: value R -> 330R
- U1: footprint DRV_8833_module:3pin_Reflection_sensor -> DRV_8833_module:IR sensor header
- U3: footprint DRV_8833_module:3pin_Reflection_sensor -> DRV_8833_module:HC-05 header
- U4: footprint DRV_8833_module:3pin_Reflection_sensor -> DRV_8833_module:OLED display header
- moved R1 98.0 mm to (120.0, 34.0), turned to -90 degrees
- moved D1 97.7 mm to (120.0, 28.0), turned to -90 degrees
- moved U1 76.3 mm to (109.3, 110.8), turned to 180 degrees
- moved U4 51.1 mm to (86.7, 29.0), turned to 90 degrees
- moved U3 28.4 mm to (110.0, 25.0)
- moved C4 17.4 mm to (64.9, 85.1), turned to 0 degrees
- moved C3 5.54 mm to (56.0, 47.1)
- moved D2 5.54 mm to (56.2, 38.3)
- moved C1 4.95 mm to (100.0, 83.4)
- moved J1 4.57 mm to (43.7, 50.0)
- moved C2 1.07 mm to (100.6, 71.1)
Connections:
- A1 pad 1: unconnected-(A1-D1/TX-Pad1) -> Ard_Tx
- A1 pad 15: Net-(A1-D12) -> unconnected-(A1-D12-Pad15)
- A1 pad 19: IR5 -> IR1
- A1 pad 2: unconnected-(A1-D0/RX-Pad2) -> Ard_Rx
- A1 pad 20: IR4 -> IR2
- A1 pad 22: IR2 -> IR4
- A1 pad 23: IR1 -> SDA
- A1 pad 24: unconnected-(A1-A5-Pad24) -> SCL
- A1 pad 25: unconnected-(A1-A6-Pad25) -> IR5
- A1 pad 7: unconnected-(A1-D4-Pad7) -> Buzzer
- A1 pad 8: unconnected-(A1-D5-Pad8) -> Blinker_L
- A1 pad 9: unconnected-(A1-D6-Pad9) -> Blinker_R
- R1 pad 2: Net-(A1-D12) -> Blinker_L
- U1 pad 2: GND -> IR1
- U1 pad 3: IR1 -> IR2
- U2 pad 2: Net-(J2-Pin_1) -> Net-(U2-OUT1)
- U2 pad 4: Net-(J3-Pin_1) -> Net-(U2-OUT3)
- U3 pad 1: +5V_MCU -> unconnected-(U3-State-Pad1)
- U3 pad 2: GND -> Net-(U3-Rx)
- U3 pad 3: IR2 -> Ard_Rx
- U4 pad 1: +5V_MCU -> GND
- U4 pad 2: GND -> +5V_MCU
- U4 pad 3: IR3 -> SCL
Routing:
- net Blinker_R: track 0.00 -> 115.3 mm, vias 0 -> 1
- net Blinker_L: track 0.00 -> 92.6 mm, vias 0 -> 1
- net SDA: track 0.00 -> 87.2 mm, vias 0 -> 2
- net SCL: track 0.00 -> 82.1 mm, vias 0 -> 2
- net +5V_bat: track 99.2 -> 171.2 mm
- net Ard_Rx: track 0.00 -> 61.7 mm, vias 0 -> 1
- net Ard_Tx: track 0.00 -> 55.4 mm, vias 0 -> 1
- net Buzzer: track 0.00 -> 43.7 mm, vias 0 -> 1
- net +5V_MCU: track 251.6 -> 212.4 mm
- net Net-(A1-D12): track 25.1 -> 0.00 mm
- net IR5: track 88.9 -> 66.1 mm
- net IR1: track 101.3 -> 80.9 mm
- net IR4: track 89.3 -> 70.2 mm
- net IR3: track 91.8 -> 73.7 mm
- net IR2: track 94.7 -> 77.3 mm
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Other:
- outline, holes or cut-outs redrawn
- board text added: "+5V_bat"
- board text added: "+5V_bat Gnd"
- board text added: "FrenGP Robotek 1.1"
- board text added: "Gnd IR5 IR4 IR3 IR2 IR1 Vcc"
- board text removed: "FrenGP Robotek 1.0"
